File: Summer_project/Summer_project.kicad_pcb (KiCad board)
At the start: 2 copper layers, 97.3 x 90.7 mm, 17 parts, among them Q3 2N3904, Q4 2N3904, SW1 SW_Push

Commit message: added_logos
Parts:
- added G***: LOGO, Summer_project:TU, B.Cu at (119.0, 62.0)
- added G***: LOGO, Summer_project:PCB_WAY_2.0, B.Cu at (119.0, 92.0)
- added G***: LOGO, Summer_project:ifixit, B.Cu at (186.0, 88.5)
- added G***: LOGO, Summer_project:RSC_for_back_silk, B.Cu at (119.0, 79.5)
- added REF**: OSHW-Logo_5.7x6mm_SilkScreen, Symbol:OSHW-Logo_5.7x6mm_SilkScreen, B.Cu at (173.0, 92.0)

Commit message: update
Parts:
- moved G*** 1.67 mm to (184.6, 89.4)
Other:
- board text added: "RSC Summer School"
- board text removed: "RSC Summer School Badge"
Changed lines of the file:
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@@
 	(footprint "Summer_project:ifixit"
 		(layer "B.Cu")
-		(at 186 88.5 180)
+		(at 184.601424 89.416608 180)
 		(property "Reference" "G***"
 			(at 6.383954 -26.282405 0)
@@
 		)
 	)
-	(gr_text "RSC Summer School Badge"
+	(gr_text "RSC Summer School"
 		(at 188 57.5 0)
 		(layer "B.SilkS")

Commit message: latest; fully reviewed, more metadata and B.silkscreen furnished; exported gerbers incl orderable zip via pcbway
Parts:
- added REF**: KiCad-Logo2_8mm_SilkScreen, Symbol:KiCad-Logo2_8mm_SilkScreen, B.Cu at (125.0, 125.8)
- moved G*** 65.0 mm to (120.1, 81.1)
- moved G*** 64.2 mm to (181.8, 66.0)
- moved REF** 11.5 mm to (163.0, 97.6)
- moved G*** 7.62 mm to (120.1, 69.5)
- moved G*** 5.13 mm to (229.8, 44.4)
- moved G*** 1.35 mm to (120.1, 92.8)
Other:
- board text added: "10u"
- board text added: "330"
- board text added: "470"
- board text added: "68k"
- board text added: "Astable Multivibrator f = 0.72/RC R=68kΩ C=10µF ~1.06Hz Based on: gitlab.com/evils/kicad-workshop"
- board text added: "CR2032 3V ~225mAh Runtime: ~20hrs (Pad = GND)"
- board text added: "Designing Social Robots for Human Interaction"
- board text added: "This badge belongs to:"
- board text added: "f = 1/(2·ln2·RC) ≈ 0.72/RC"
- board text removed: "Name:"
- board text removed: "RSC Summer School"
